File: PCBPT_V2/Hardware/StepperMotor_module/Motor_module.kicad_pcb (KiCad board)
At the start: 2 copper layers, 28.5 x 40 mm, 34 parts, among them J1 Limit Switch, J2 Limit Switch, J3 Limit Switch, J4 Limit Switch, J5 Conn_01x08_Male, J6 Conn_01x04_Male, J7 Conn_01x08_Female, J8 Conn_01x08_Female, SW1 SW_Push, U1 STM32F031F6Px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

Commit message: udated by FZ
Other:
- board text added: "Coral"
- board text removed: "Polyp"
Changed lines of the file:
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@@
     (effects (font (size 1 1) (thickness 0.15)) (justify mirror))
   )
-  (gr_text "Polyp" (at 156.7 91.85) (layer "B.SilkS")
+  (gr_text "Coral" (at 155.829991 91.850007) (layer "B.SilkS")
     (effects (font (size 1.7 1.7) (thickness 0.3)) (justify mirror))
   )
-  (gr_text "Stepper V1.0" (at 146.7 92.3) (layer "B.SilkS")
+  (gr_text "Stepper V1.0" (at 145.830009 92.3) (layer "B.SilkS")
     (effects (font (size 1.1 1.1) (thickness 0.18)) (justify mirror))
   )
