File: PCBPT_V2/Hardware/StepperMotor_module/Motor_module.kicad_sch (KiCad schematic)
At the start: 34 parts, among them J1 Limit Switch, J2 Limit Switch, J3 Limit Switch, J4 Limit Switch, J5 Conn_01x08_Male, J6 Conn_01x04_Male, J7 Conn_01x08_Female, J8 Conn_01x08_Female, SW1 SW_Push, U1 STM32F031F6Px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

Commit message: udated by FZ
Parts:
- C1: value (none) -> 100uF; footprint (none) -> Capacitor_THT:CP_Radial_D5.0mm_P2.50mm
- SW1: footprint (none) -> Button_Switch_SMD:SW_Push_1P1T_NO_CK_KMR2
Other:
- moved on the sheet: D2, D3, J1, J2, J3, J4, J5, R10, R9

Commit message: udated by FZ
Parts:
- U1: value STM32F031F6Px -> (none)
Changed lines of the file:
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@@
       (effects (font (size 1.27 1.27)) (justify left))
     )
-    (property "Value" "STM32F031F6Px" (id 1) (at 49.53 57.15 90)
+    (property "Value" "" (id 1) (at 49.53 57.15 90)
       (effects (font (size 1.27 1.27)) (justify left))
     )

Commit message: udated by FZ
Parts:
- U1: value (none) -> STM32F031F6Px
