File: PCBPT_V2/Hardware/StepperMotor_module_V2_XIAO_RP2040/StepperMotor_module_V2_XIAO_RP2040.kicad_pcb (KiCad board)
At the start: 2 copper layers, 43 x 31.5 mm, 25 parts, among them J3 Servo, J4 Limit Switch, J5 Conn_01x09_Pin, J6 Limit Switch, J7 Limit Switch, U1 MOUDLE-SEEEDUINO-XIAO

Commit message: udated by FZ
Changed lines of the file:
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@@
   (segment (start 149.4775 71.84) (end 149.4875 71.85) (width 0.254) (layer "F.Cu") (net 8))
   (segment (start 145.8 71.84) (end 149.4775 71.84) (width 0.254) (layer "F.Cu") (net 8))
-  (segment (start 145.8 79.46) (end 143.63 79.46) (width 0.254) (layer "F.Cu") (net 9))
+  (segment (start 127.70975 80.15) (end 145.11 80.15) (width 0.254) (layer "F.Cu") (net 9))
+  (segment (start 145.11 80.15) (end 145.8 79.46) (width 0.254) (layer "F.Cu") (net 9))
   (segment (start 125.39925 82.4605) (end 127.70975 80.15) (width 0.254) (layer "F.Cu") (net 9))
-  (segment (start 142.94 80.15) (end 140.7 80.15) (width 0.254) (layer "F.Cu") (net 9))
-  (segment (start 127.70975 80.15) (end 140.7 80.15) (width 0.254) (layer "F.Cu") (net 9))
-  (segment (start 143.63 79.46) (end 142.94 80.15) (width 0.254) (layer "F.Cu") (net 9))
   (segment (start 144.45 80.65) (end 145.8 82) (width 0.254) (layer "F.Cu") (net 10))
   (segment (start 127.93925 82.4605) (end 129.74975 80.65) (width 0.254) (layer "F.Cu") (net 10))
