File: PCBPT_V2/Hardware/StepperMotor_module_V2_XIAO_RP2040/StepperMotor_module_V2_XIAO_RP2040.kicad_sch (KiCad schematic)
At the start: 0 parts

Commit message: udated by FZ
Other:
- added sheet A4988_Module (A4988_Module.kicad_sch)
- added sheet Conn (conn.kicad_sch)
Changed lines of the file:
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@@
+    )
+  )
+  (sheet (at 40.64 39.37) (size 30.48 8.89) (fields_autoplaced)
+    (stroke (width 0.1524) (type solid))
+    (fill (color 0 0 0 0.0000))
+    (property "Sheetname" "Conn" (at 40.64 38.6584 0) (show_name)
+      (effects (font (size 1.27 1.27) bold italic) (justify left bottom))
+    )
+    (property "Sheetfile" "conn.kicad_sch" (at 40.64 48.8446 0) (show_name)
+      (effects (font (size 1.27 1.27) bold italic) (justify left top))
+    )
+    (instances
+      (project "StepperMotor_module_V2_XIAO_RP2040"
+        (path "/67ad53b0-e724-4354-8add-ffbe056bca93" (page "4"))
+      )
+    )
+  )
+  (sheet (at 76.2 22.86) (size 31.75 8.89) (fields_autoplaced)
+    (stroke (width 0.1524) (type solid))
+    (fill (color 0 0 0 0.0000))
+    (property "Sheetname" "A4988_Module" (at 76.2 22.1484 0) (show_name)
+      (effects (font (size 1.27 1.27) bold italic) (justify left bottom))
+    )
+    (property "Sheetfile" "A4988_Module.kicad_sch" (at 76.2 32.3346 0) (show_name)
+      (effects (font (size 1.27 1.27) bold italic) (justify left top))
+    )
+    (instances
+      (project "StepperMotor_module_V2_XIAO_RP2040"
+        (path "/67ad53b0-e724-4354-8add-ffbe056bca93" (page "3"))
+      )
     )
   )
