File: PCBPT_V2/Hardware/StepperMotor_module_V2_XIAO_RP2040_w_PWR/StepperMotor_module_V2_XIAO_RP2040.kicad_pcb (KiCad board)
At the start: 2 copper layers, 43 x 31.5 mm, 25 parts, among them J3 Servo, J4 Limit Switch, J5 Conn_01x09_Pin, J6 Limit Switch, J7 Limit Switch, U1 MOUDLE-SEEEDUINO-XIAO

Commit message: udated by FZ
Parts:
- removed J5: Conn_01x09_Pin, Connector_PinHeader_2.54mm:PinHeader_1x09_P2.54mm_Vertical
- added C4: 0.47uF, Capacitor_SMD:C_0805_2012Metric_Pad1.18x1.45mm_HandSolder, B.Cu at (140.4, 79.3)
- added C5: 0.1uF, Capacitor_SMD:C_0805_2012Metric_Pad1.18x1.45mm_HandSolder, B.Cu at (130.5, 62.8)
- added IC1: LM2940IMP-5.0_NOPB, SamacSys_Parts:SOT230P700X180-4N, B.Cu at (139.2, 73.8)
- added J1: Conn_01x08_Pin, Connector_PinHeader_2.54mm:PinHeader_1x08_P2.54mm_Vertical, F.Cu at (153.8, 87.5)
- C3: value 0.1uF -> 22uF
- moved C3 15.7 mm to (134.0, 77.0)
- moved D1 1.40 mm to (161.6, 81.4), turned to 90 degrees
- moved R8 0.87 mm to (163.2, 81.4), turned to 90 degrees
Routing:
- net VPP: track 31.3 -> 47.9 mm
- net VCC: track 60.8 -> 66.8 mm, vias 1 -> 2
- net SDA: track 7.60 -> 10.1 mm
- net GPIO: track 7.60 -> 10.1 mm
- net SCL: track 7.60 -> 10.1 mm
- net GND: vias 41 -> 42

Commit message: udated by FZ
Parts:
- J1: moved to B.Cu
- turned J1 to 90 degrees
Changed lines of the file:
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@@
-    )
-  )
-  (footprint "Connector_PinHeader_2.54mm:PinHeader_1x08_P2.54mm_Vertical" (layer "F.Cu")
-    (at 153.78 87.5 -90)
-    (descr "Through hole straight pin header, 1x08, 2.54mm pitch, single row")
-    (tags "Through hole pin header THT 1x08 2.54mm single row")
-    (property "Sheetfile" "conn.kicad_sch")
-    (property "Sheetname" "Conn")
-    (property "ki_description" "Generic connector, single row, 01x08, script generated")
-    (property "ki_keywords" "connector")
-    (attr through_hole)
-    (fp_text reference "J1" (at 0 -2.33 90) (layer "F.SilkS") hide
-        (effects (font (size 1 1) (thickness 0.15)))
-    )
-    (fp_text value "Conn_01x08_Pin" (at 0 20.11 90) (layer "F.Fab")
-        (effects (font (size 1 1) (thickness 0.15)))
-    )
-    (fp_text user "${REFERENCE}" (at 0 8.89) (layer "F.Fab")
-        (effects (font (size 1 1) (thickness 0.15)))
-    )
-    (fp_line (start -1.33 -1.33) (end 0 -1.33)
-      (stroke (width 0.12) (type solid)) (layer "F.SilkS"))
-    (fp_line (start -1.33 0) (end -1.33 -1.33)
-      (stroke (width 0.12) (type solid)) (layer "F.SilkS"))
-    (fp_line (start -1.33 1.27) (end -1.33 19.11)
-      (stroke (width 0.12) (type solid)) (layer "F.SilkS"))
-    (fp_line (start -1.33 1.27) (end 1.33 1.27)
-      (stroke (width 0.12) (type solid)) (layer "F.SilkS"))
-    (fp_line (start -1.33 19.11) (end 1.33 19.11)
-      (stroke (width 0.12) (type solid)) (layer "F.SilkS"))
-    (fp_line (start 1.33 1.27) (end 1.33 19.11)
-      (stroke (width 0.12) (type solid)) (layer "F.SilkS"))
-    (fp_line (start -1.8 -1.8) (end -1.8 19.55)
-      (stroke (width 0.05) (type solid)) (layer "F.CrtYd"))
-    (fp_line (start -1.8 19.55) (end 1.8 19.55)
-      (stroke (width 0.05) (type solid)) (layer "F.CrtYd"))
-    (fp_line (start 1.8 -1.8) (end -1.8 -1.8)
-      (stroke (width 0.05) (type solid)) (layer "F.CrtYd"))
-    (fp_line (start 1.8 19.55) (end 1.8 -1.8)
-      (stroke (width 0.05) (type solid)) (layer "F.CrtYd"))
-    (fp_line (start -1.27 -0.635) (end -0.635 -1.27)
-      (stroke (width 0.1) (type solid)) (layer "F.Fab"))
-    (fp_line (start -1.27 19.05) (end -1.27 -0.635)
-      (stroke (width 0.1) (type solid)) (layer "F.Fab"))
-    (fp_line (start -0.635 -1.27) (end 1.27 -1.27)
-      (stroke (width 0.1) (type solid)) (layer "F.Fab"))
-    (fp_line (start 1.27 -1.27) (end 1.27 19.05)
-      (stroke (width 0.1) (type solid)) (layer "F.Fab"))
-    (fp_line (start 1.27 19.05) (end -1.27 19.05)
-      (stroke (width 0.1) (type solid)) (layer "F.Fab"))
-    (pad "1" thru_hole rect (at 0 0 270) (size 1.7 1.7) (drill 1) (layers "*.Cu" "*.Mask")
-      (net 2 "VPP") (pinfunction "Pin_1") (pintype "passive"))
-    (pad "2" thru_hole oval (at 0 2.54 270) (size 1.7 1.7) (drill 1) (layers "*.Cu" "*.Mask")
-      (net 2 "VPP") (pinfunction "Pin_2") (pintype "passive"))
-    (pad "3" thru_hole oval (at 0 5.08 270) (size 1.7 1.7) (drill 1) (layers "*.Cu" "*.Mask")
-      (net 23 "GPIO") (pinfunction "Pin_3") (pintype "passive"))
-    (pad "4" thru_hole oval (at 0 7.62 270) (size 1.7 1.7) (drill 1) (layers "*.Cu" "*.Mask")
-      (net 19 "SCL") (pinfunction "Pin_4") (pintype "passive"))
-    (pad "5" thru_hole oval (at 0 10.16 270) (size 1.7 1.7) (drill 1) (layers "*.Cu" "*.Mask")
-      (net 20 "SDA") (pinfunction "Pin_5") (pintype "passive"))
-    (pad "6" thru_hole oval (at 0 12.7 270) (size 1.7 1.7) (drill 1) (layers "*.Cu" "*.Mask")
-      (net 1 "GND") (pinfunction "Pin_6") (pintype "passive"))
-    (pad "7" thru_hole oval (at 0 15.24 270) (size 1.7 1.7) (drill 1) (layers "*.Cu" "*.Mask")
-      (net 1 "GND") (pinfunction "Pin_7") (pintype "passive"))
-    (pad "8" thru_hole oval (at 0 17.78 270) (size 1.7 1.7) (drill 1) (layers "*.Cu" "*.Mask")
-      (net 1 "GND") (pinfunction "Pin_8") (pintype "passive"))
-    (model "${KICAD6_3DMODEL_DIR}/Connector_PinHeader_2.54mm.3dshapes/PinHeader_1x08_P2.54mm_Vertical.wrl"
-      (offset (xyz 0 0 0))
-      (scale (xyz 1 1 1))
-      (rotate (xyz 0 0 0))
     )
   )
@@
       (offset (xyz 0 0 0))
       (scale (xyz 1 1 1))
+      (rotate (xyz 0 0 0))
+    )
+  )
+  (footprint "Connector_PinHeader_2.54mm:PinHeader_1x08_P2.54mm_Vertical" (layer "B.Cu")
+    (at 153.765 87.5 90)
+    (descr "Through hole straight pin header, 1x08, 2.54mm pitch, single row")
+    (tags "Through hole pin header THT 1x08 2.54mm single row")
+    (property "Sheetfile" "conn.kicad_sch")
+    (property "Sheetname" "Conn")
+    (property "ki_description" "Generic connector, single row, 01x08, script generated")
+    (property "ki_keywords" "connector")
+    (attr through_hole)
+    (fp_text reference "J1" (at 0 2.33 90) (layer "B.SilkS") hide
+        (effects (font (size 1 1) (thickness 0.15)) (justify mirror))
+    )
+    (fp_text value "Conn_01x08_Pin" (at 0 -20.11 90) (layer "B.Fab")
+        (effects (font (size 1 1) (thickness 0.15)) (justify mirror))
+    )
+    (fp_text user "${REFERENCE}" (at 0 -8.89) (layer "B.Fab")
+        (effects (font (size 1 1) (thickness 0.15)) (justify mirror))
+    )
+    (fp_line (start -1.33 -19.11) (end 1.33 -19.11)
+      (stroke (width 0.12) (type solid)) (layer "B.SilkS"))
+    (fp_line (start -1.33 -1.27) (end -1.33 -19.11)
+      (stroke (width 0.12) (type solid)) (layer "B.SilkS"))
+    (fp_line (start -1.33 -1.27) (end 1.33 -1.27)
+      (stroke (width 0.12) (type solid)) (layer "B.SilkS"))
+    (fp_line (start -1.33 0) (end -1.33 1.33)
+      (stroke (width 0.12) (type solid)) (layer "B.SilkS"))
+    (fp_line (start -1.33 1.33) (end 0 1.33)
+      (stroke (width 0.12) (type solid)) (layer "B.SilkS"))
+    (fp_line (start 1.33 -1.27) (end 1.33 -19.11)
+      (stroke (width 0.12) (type solid)) (layer "B.SilkS"))
+    (fp_line (start -1.8 -19.55) (end 1.8 -19.55)
+      (stroke (width 0.05) (type solid)) (layer "B.CrtYd"))
+    (fp_line (start -1.8 1.8) (end -1.8 -19.55)
+      (stroke (width 0.05) (type solid)) (layer "B.CrtYd"))
+    (fp_line (start 1.8 -19.55) (end 1.8 1.8)
+      (stroke (width 0.05) (type solid)) (layer "B.CrtYd"))
+    (fp_line (start 1.8 1.8) (end -1.8 1.8)
+      (stroke (width 0.05) (type solid)) (layer "B.CrtYd"))
+    (fp_line (start -1.27 -19.05) (end -1.27 0.635)
+      (stroke (width 0.1) (type solid)) (layer "B.Fab"))
+    (fp_line (start -1.27 0.635) (end -0.635 1.27)
+      (stroke (width 0.1) (type solid)) (layer "B.Fab"))
+    (fp_line (start -0.635 1.27) (end 1.27 1.27)
+      (stroke (width 0.1) (type solid)) (layer "B.Fab"))
+    (fp_line (start 1.27 -19.05) (end -1.27 -19.05)
+      (stroke (width 0.1) (type solid)) (layer "B.Fab"))
+    (fp_line (start 1.27 1.27) (end 1.27 -19.05)
+      (stroke (width 0.1) (type solid)) (layer "B.Fab"))
+    (pad "1" thru_hole rect (at 0 0 90) (size 1.7 1.7) (drill 1) (layers "*.Cu" "*.Mask")
+      (net 2 "VPP") (pinfunction "Pin_1") (pintype "passive"))
+    (pad "2" thru_hole oval (at 0 -2.54 90) (size 1.7 1.7) (drill 1) (layers "*.Cu" "*.Mask")
+      (net 2 "VPP") (pinfunction "Pin_2") (pintype "passive"))
+    (pad "3" thru_hole oval (at 0 -5.08 90) (size 1.7 1.7) (drill 1) (layers "*.Cu" "*.Mask")
+      (net 23 "GPIO") (pinfunction "Pin_3") (pintype "passive"))
+    (pad "4" thru_hole oval (at 0 -7.62 90) (size 1.7 1.7) (drill 1) (layers "*.Cu" "*.Mask")
+      (net 19 "SCL") (pinfunction "Pin_4") (pintype "passive"))
+    (pad "5" thru_hole oval (at 0 -10.16 90) (size 1.7 1.7) (drill 1) (layers "*.Cu" "*.Mask")
+      (net 20 "SDA") (pinfunction "Pin_5") (pintype "passive"))
+    (pad "6" thru_hole oval (at 0 -12.7 90) (size 1.7 1.7) (drill 1) (layers "*.Cu" "*.Mask")
+      (net 1 "GND") (pinfunction "Pin_6") (pintype "passive"))
+    (pad "7" thru_hole oval (at 0 -15.24 90) (size 1.7 1.7) (drill 1) (layers "*.Cu" "*.Mask")
+      (net 1 "GND") (pinfunction "Pin_7") (pintype "passive"))
+    (pad "8" thru_hole oval (at 0 -17.78 90) (size 1.7 1.7) (drill 1) (layers "*.Cu" "*.Mask")
+      (net 1 "GND") (pinfunction "Pin_8") (pintype "passive"))
+    (model "${KICAD6_3DMODEL_DIR}/Connector_PinHeader_2.54mm.3dshapes/PinHeader_1x08_P2.54mm_Vertical.wrl"
+      (offset (xyz 0 0 0))
+      (scale (xyz 1 1 1))
