File: PCBPT_V2/Hardware/StepperMotor_module_V2_XIAO_RP2040_w_PWR/Power.kicad_sch (KiCad schematic)
At the start: 4 parts, among them IC1 LM2940IMP-5.0_NOPB

Commit message: udated by FZ
Changed lines of the file:
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@@
   (symbol (lib_id "SamacSys_Parts:LM2940IMP-5.0_NOPB") (at 66.04 43.18 0) (unit 1)
     (in_bom yes) (on_board yes) (dnp no) (fields_autoplaced)
-    (property "Reference" "IC1" (at 81.28 37.1108 0)
+    (property "Reference" "IC1" (at 78.74 37.1108 0)
       (effects (font (size 1.27 1.27)))
     )
-    (property "Value" "LM2940IMP-5.0_NOPB" (at 81.28 39.1588 0)
+    (property "Value" "LM2940IMP-5.0_NOPB" (at 78.74 39.1588 0)
       (effects (font (size 1.27 1.27)))
     )

Commit message: udated by FZ
Parts:
- IC1: value LM2940IMP-5.0_NOPB -> UA78M05IDCYR
Changed lines of the file:
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@@
       (effects (font (size 1.27 1.27)))
     )
-    (property "Value" "LM2940IMP-5.0_NOPB" (at 78.74 39.1588 0)
+    (property "Value" "UA78M05IDCYR" (at 78.74 39.1588 0)
       (effects (font (size 1.27 1.27)))
     )
