File: PCBPT_V2/Hardware/RPi_Pico_W_A4988_control_board/A4988_Module.kicad_sch (KiCad schematic)
At the start: 42 parts, among them J13 Conn_02x03_Odd_Even, J14 Conn_02x03_Odd_Even, J15 Conn_02x03_Odd_Even, J16 Conn_02x03_Odd_Even, J17 Conn_02x03_Odd_Even, J18 Conn_02x03_Odd_Even

Commit message: udated by FZ
Parts:
- removed R6 (x18): 10K, Resistor_SMD:R_0603_1608Metric_Pad0.98x0.95mm_HandSolder, symbol Device:R_Small
- added A7, A8: Pololu_Breakout_A4988, Module:Pololu_Breakout-16_15.2x20.3mm, symbol Driver_Motor:Pololu_Breakout_A4988
- added C11 (x2): 100uF, Capacitor_THT:CP_Radial_D6.3mm_P2.50mm, symbol Device:C_Polarized_Small
- added J24, J25: Conn_02x03_Odd_Even, Connector_PinHeader_2.54mm:PinHeader_2x03_P2.54mm_Vertical, symbol Connector_Generic:Conn_02x03_Odd_Even
- added R6 (x2): 10K, Resistor_SMD:R_1206_3216Metric_Pad1.30x1.75mm_HandSolder, symbol Device:R_Small
- C11: footprint (none) -> Capacitor_THT:CP_Radial_D6.3mm_P2.50mm
- J13, J14, J15, J16, J17, J18: footprint (none) -> Connector_PinHeader_2.54mm:PinHeader_2x03_P2.54mm_Vertical
- R6: footprint Resistor_SMD:R_0603_1608Metric_Pad0.98x0.95mm_HandSolder -> Resistor_SMD:R_1206_3216Metric_Pad1.30x1.75mm_HandSolder
Connections:
- net +3V3: now also J13.2 (Pin_2), J13.4 (Pin_4), J13.6 (Pin_6), J14.2 (Pin_2), J14.4 (Pin_4), J14.6 (Pin_6), J15.2 (Pin_2), J15.4 (Pin_4), J15.6 (Pin_6), J16.2 (Pin_2), J16.4 (Pin_4), J16.6 (Pin_6), J17.2 (Pin_2), J17.4 (Pin_4), J17.6 (Pin_6), J18.2 (Pin_2), J18.4 (Pin_4), J18.6 (Pin_6), A7.2 (VDD), A8.2 (VDD), J24.2 (Pin_2), J24.4 (Pin_4), J24.6 (Pin_6), J25.2 (Pin_2), J25.4 (Pin_4), J25.6 (Pin_6)
- net GND: now also A7.1 (GND), A7.7 (GND), A8.1 (GND), A8.7 (GND), C11.2, C11.2, R6.2, R6.2; no longer J13.1 (Pin_1), J13.3 (Pin_3), J13.5 (Pin_5), J14.1 (Pin_1), J14.3 (Pin_3), J14.5 (Pin_5), J15.1 (Pin_1), J15.3 (Pin_3), J15.5 (Pin_5), J16.1 (Pin_1), J16.3 (Pin_3), J16.5 (Pin_5), J17.1 (Pin_1), J17.3 (Pin_3), J17.5 (Pin_5), J18.1 (Pin_1), J18.3 (Pin_3), J18.5 (Pin_5)
- net MS1_1: now also J13.1 (Pin_1); no longer J13.2 (Pin_2)
- net MS1_2: now also J14.1 (Pin_1); no longer J14.2 (Pin_2)
- net MS1_3: now also J15.1 (Pin_1); no longer J15.2 (Pin_2)
- net MS1_4: now also J16.1 (Pin_1); no longer J16.2 (Pin_2)
- net MS1_5: now also J17.1 (Pin_1); no longer J17.2 (Pin_2)
- net MS1_6: now also J18.1 (Pin_1); no longer J18.2 (Pin_2)
- net MS2_1: now also J13.3 (Pin_3); no longer J13.4 (Pin_4)
- net MS2_2: now also J14.3 (Pin_3); no longer J14.4 (Pin_4)
- net MS2_3: now also J15.3 (Pin_3); no longer J15.4 (Pin_4)
- net MS2_4: now also J16.3 (Pin_3); no longer J16.4 (Pin_4)
- net MS2_5: now also J17.3 (Pin_3); no longer J17.4 (Pin_4)
- net MS2_6: now also J18.3 (Pin_3); no longer J18.4 (Pin_4)
- net MS3_1: now also J13.5 (Pin_5); no longer J13.6 (Pin_6)
- net MS3_2: now also J14.5 (Pin_5); no longer J14.6 (Pin_6)
- net MS3_3: now also J15.5 (Pin_5); no longer J15.6 (Pin_6)
- net MS3_4: now also J16.5 (Pin_5); no longer J16.6 (Pin_6)
- net MS3_5: now also J17.5 (Pin_5); no longer J17.6 (Pin_6)
- net MS3_6: now also J18.5 (Pin_5); no longer J18.6 (Pin_6)
- net VPP: now also A7.8 (VMOT), A8.8 (VMOT), C11.1, C11.1
- new net: A8.13 (~{RESET}), A8.14 (~{SLEEP})
- new net: A8.9 (~{ENABLE}), R6.1
- new net: A7.13 (~{RESET}), A7.14 (~{SLEEP})
- new net: A7.9 (~{ENABLE}), R6.1
- new net 1A_7: A7.4 (1A)
- new net 1A_8: A8.4 (1A)
- new net 1B_7: A7.3 (1B)
- new net 1B_8: A8.3 (1B)
- new net 2A_7: A7.5 (2A)
- new net 2A_8: A8.5 (2A)
- new net 2B_7: A7.6 (2B)
- new net 2B_8: A8.6 (2B)
- new net DIR_7: A7.16 (DIR)
- new net DIR_8: A8.16 (DIR)
- new net MS1_7: A7.10 (MS1), J24.1 (Pin_1)
- new net MS1_8: A8.10 (MS1), J25.1 (Pin_1)
- new net MS2_7: A7.11 (MS2), J24.3 (Pin_3)
- new net MS2_8: A8.11 (MS2), J25.3 (Pin_3)
- new net MS3_7: A7.12 (MS3), J24.5 (Pin_5)
- new net MS3_8: A8.12 (MS3), J25.5 (Pin_5)
- new net STEP_7: A7.15 (STEP)
- new net STEP_8: A8.15 (STEP)
Other:
- moved on the sheet: J13, J14, J15, J16, J17, J18
