File: PCBPT_V2/Hardware/RPi_Pico_W_A4988_control_board/Power.kicad_sch (KiCad schematic)
At the start: 6 parts, among them IC1 UA78M05IDCYR

Commit message: udated by FZ
Parts:
- added J30, J31: pin, Mylib:conn_SMD_15mmx5mm, symbol Mylib:pin
- added U1: 3544-2, SamacSys_Parts:3544-2, symbol SamacSys_Parts:3544-2
- C11: footprint (none) -> Capacitor_THT:CP_Radial_D12.5mm_P5.00mm
- C2: footprint Capacitor_SMD:C_0805_2012Metric_Pad1.18x1.45mm_HandSolder -> Capacitor_SMD:C_1206_3216Metric_Pad1.33x1.80mm_HandSolder
- R38: footprint (none) -> Resistor_SMD:R_1206_3216Metric_Pad1.30x1.75mm_HandSolder
Connections:
- net +12V: now also J30.1, U1.1, U1.2; no longer C2.1, IC1.1 (IN), R38.1
- net GND: now also J31.1
- new net VPP: C2.1, IC1.1 (IN), R38.1, U1.3, U1.4
Other:
- moved on the sheet: C11, R38
