File: PCBPT_V2/Hardware/RPi_Pico_W_A4988_control_board/RPi_Pico_W_A4988_control_board.kicad_pcb (KiCad board)
At the start: 2 copper layers, 0 parts

Commit message: udated by FZ
Parts:
- added A1: Pololu_Breakout_A4988, Module:Pololu_Breakout-16_15.2x20.3mm, F.Cu at (160.6, 121.9)
- added A2: Pololu_Breakout_A4988, Module:Pololu_Breakout-16_15.2x20.3mm, F.Cu at (183.5, 121.9)
- added A3: Pololu_Breakout_A4988, Module:Pololu_Breakout-16_15.2x20.3mm, F.Cu at (183.5, 98.2)
- added A4: Pololu_Breakout_A4988, Module:Pololu_Breakout-16_15.2x20.3mm, F.Cu at (160.6, 98.2)
- added A5: Pololu_Breakout_A4988, Module:Pololu_Breakout-16_15.2x20.3mm, F.Cu at (183.5, 74.5)
- added A6: Pololu_Breakout_A4988, Module:Pololu_Breakout-16_15.2x20.3mm, F.Cu at (160.6, 74.6)
- added A7: Pololu_Breakout_A4988, Module:Pololu_Breakout-16_15.2x20.3mm, F.Cu at (160.6, 50.9)
- added A8: Pololu_Breakout_A4988, Module:Pololu_Breakout-16_15.2x20.3mm, F.Cu at (183.5, 50.9)
- added C1: 0.01uF, Capacitor_SMD:C_1206_3216Metric_Pad1.33x1.80mm_HandSolder, F.Cu at (132.8, 53.1)
- added C10: 0.01uF, Capacitor_SMD:C_1206_3216Metric_Pad1.33x1.80mm_HandSolder, F.Cu at (114.5, 88.5)
- added C11: 470uF, Capacitor_THT:CP_Radial_D12.5mm_P5.00mm, F.Cu at (109.4, 48.2)
- added C12: 100uF, Capacitor_THT:CP_Radial_D6.3mm_P2.50mm, F.Cu at (155.2, 37.9)
- added C13: 100uF, Capacitor_THT:CP_Radial_D6.3mm_P2.50mm, F.Cu at (178.0, 38.0)
- added C14: 100uF, Capacitor_THT:CP_Radial_D6.3mm_P2.50mm, F.Cu at (178.0, 62.0)
- added C15: 100uF, Capacitor_THT:CP_Radial_D6.3mm_P2.50mm, F.Cu at (178.0, 85.5)
- added C16: 100uF, Capacitor_THT:CP_Radial_D6.3mm_P2.50mm, F.Cu at (155.2, 85.5)
- added C17: 100uF, Capacitor_THT:CP_Radial_D6.3mm_P2.50mm, F.Cu at (155.2, 62.0)
- added C18: 100uF, Capacitor_THT:CP_Radial_D6.3mm_P2.50mm, F.Cu at (155.2, 108.9)
- added C19: 100uF, Capacitor_THT:CP_Radial_D6.3mm_P2.50mm, F.Cu at (178.0, 109.0)
- added C2: 0.01uF, Capacitor_SMD:C_1206_3216Metric_Pad1.33x1.80mm_HandSolder, F.Cu at (123.9, 53.1)
- added C3: 22uF, Capacitor_SMD:C_1206_3216Metric_Pad1.33x1.80mm_HandSolder, F.Cu at (107.3, 113.2)
- added C4: 0.47uF, Capacitor_SMD:C_1206_3216Metric_Pad1.33x1.80mm_HandSolder, F.Cu at (106.1, 107.7)
- added C5: 0.1uF, Capacitor_SMD:C_1206_3216Metric_Pad1.33x1.80mm_HandSolder, F.Cu at (107.3, 115.7)
- added C6: 0.01uF, Capacitor_SMD:C_1206_3216Metric_Pad1.33x1.80mm_HandSolder, F.Cu at (141.7, 53.1)
- added C7: 0.01uF, Capacitor_SMD:C_1206_3216Metric_Pad1.33x1.80mm_HandSolder, F.Cu at (124.0, 65.6)
- added C8: 0.01uF, Capacitor_SMD:C_1206_3216Metric_Pad1.33x1.80mm_HandSolder, F.Cu at (132.8, 65.7)
- added C9: 0.01uF, Capacitor_SMD:C_1206_3216Metric_Pad1.33x1.80mm_HandSolder, F.Cu at (141.7, 65.7)
- added D2: Schottky, Diode_SMD:D_0805_2012Metric_Pad1.15x1.40mm_HandSolder, F.Cu at (111.4, 116.7)
- added D4: LED_Small_Filled, LED_SMD:LED_1206_3216Metric_Pad1.42x1.75mm_HandSolder, F.Cu at (138.0, 41.1)
- added H1: M2, MountingHole:MountingHole_2.2mm_M2_ISO7380_Pad, F.Cu at (104.5, 31.0)
- added H2: M2, MountingHole:MountingHole_2.2mm_M2_ISO7380_Pad, F.Cu at (188.8, 31.0)
- added H3: M2, MountingHole:MountingHole_2.2mm_M2_ISO7380_Pad, F.Cu at (104.5, 123.0)
- added H4: M2, MountingHole:MountingHole_2.2mm_M2_ISO7380_Pad, F.Cu at (188.8, 123.0)
- added IC1: UA78M05IDCYR, SamacSys_Parts:SOT230P700X180-4N, F.Cu at (112.1, 108.4)
- added IC2: RASPBERRY_PI_PICO_W, SamacSys_Parts:RASPBERRYPIPICOW, F.Cu at (130.5, 99.9)
- added J1: Limit Switch, Connector_PinHeader_2.54mm:PinHeader_1x04_P2.54mm_Vertical, F.Cu at (188.2, 109.2)
- added J10: Limit Switch, Connector_PinHeader_2.54mm:PinHeader_1x02_P2.54mm_Vertical, F.Cu at (120.3, 61.1)
- added J11: Limit Switch, Connector_PinHeader_2.54mm:PinHeader_1x02_P2.54mm_Vertical, F.Cu at (129.2, 61.1)
- added J12: Limit Switch, Connector_PinHeader_2.54mm:PinHeader_1x02_P2.54mm_Vertical, F.Cu at (138.1, 61.1)
- added J13: Conn_02x03_Odd_Even, Connector_PinHeader_2.54mm:PinHeader_2x03_P2.54mm_Vertical, F.Cu at (156.8, 119.0)
- added J14: Conn_02x03_Odd_Even, Connector_PinHeader_2.54mm:PinHeader_2x03_P2.54mm_Vertical, F.Cu at (179.7, 119.0)
- added J15: Conn_02x03_Odd_Even, Connector_PinHeader_2.54mm:PinHeader_2x03_P2.54mm_Vertical, F.Cu at (179.7, 95.4)
- added J16: Conn_02x03_Odd_Even, Connector_PinHeader_2.54mm:PinHeader_2x03_P2.54mm_Vertical, F.Cu at (156.8, 95.4)
- added J17: Conn_02x03_Odd_Even, Connector_PinHeader_2.54mm:PinHeader_2x03_P2.54mm_Vertical, F.Cu at (179.7, 71.7)
- added J18: Conn_02x03_Odd_Even, Connector_PinHeader_2.54mm:PinHeader_2x03_P2.54mm_Vertical, F.Cu at (156.8, 71.7)
- added J19: Limit Switch, Connector_PinHeader_2.54mm:PinHeader_1x04_P2.54mm_Vertical, F.Cu at (104.5, 81.7)
- added J2: Limit Switch, Connector_PinHeader_2.54mm:PinHeader_1x04_P2.54mm_Vertical, F.Cu at (188.2, 85.5)
- added J20: Conn_01x06_Pin, Connector_PinHeader_2.54mm:PinHeader_1x06_P2.54mm_Vertical, F.Cu at (104.5, 61.2)
- added J21: Conn_01x06_Pin, Connector_PinHeader_2.54mm:PinHeader_1x06_P2.54mm_Vertical, F.Cu at (108.1, 61.2)
- added J22: Limit Switch, Connector_PinHeader_2.54mm:PinHeader_1x02_P2.54mm_Vertical, F.Cu at (114.7, 117.7)
- added J23: Limit Switch, Connector_PinHeader_2.54mm:PinHeader_1x02_P2.54mm_Vertical, F.Cu at (104.5, 95.0)
- added J24: Conn_02x03_Odd_Even, Connector_PinHeader_2.54mm:PinHeader_2x03_P2.54mm_Vertical, F.Cu at (156.8, 48.1)
- added J25: Conn_02x03_Odd_Even, Connector_PinHeader_2.54mm:PinHeader_2x03_P2.54mm_Vertical, F.Cu at (179.7, 48.0)
- added J26: Limit Switch, Connector_PinHeader_2.54mm:PinHeader_1x04_P2.54mm_Vertical, F.Cu at (188.2, 38.2)
- added J27: Limit Switch, Connector_PinHeader_2.54mm:PinHeader_1x04_P2.54mm_Vertical, F.Cu at (165.5, 38.2)
- added J28: Conn_01x03_Pin, Connector_PinHeader_2.54mm:PinHeader_1x03_P2.54mm_Vertical, F.Cu at (113.2, 60.1)
- added J29: Conn_01x03_Pin, Connector_PinHeader_2.54mm:PinHeader_1x03_P2.54mm_Vertical, F.Cu at (113.2, 68.8)
- added J3: Limit Switch, Connector_PinHeader_2.54mm:PinHeader_1x04_P2.54mm_Vertical, F.Cu at (165.2, 85.5)
- added J30: pin, Mylib:conn_SMD_15mmx5mm, B.Cu at (109.5, 41.0)
- added J31: pin, Mylib:conn_SMD_15mmx5mm, F.Cu at (108.5, 39.5)
- added J4: Limit Switch, Connector_PinHeader_2.54mm:PinHeader_1x04_P2.54mm_Vertical, F.Cu at (165.2, 109.2)
- added J5: Limit Switch, Connector_PinHeader_2.54mm:PinHeader_1x04_P2.54mm_Vertical, F.Cu at (188.2, 61.8)
- added J6: Limit Switch, Connector_PinHeader_2.54mm:PinHeader_1x02_P2.54mm_Vertical, F.Cu at (120.3, 48.7)
- added J7: Limit Switch, Connector_PinHeader_2.54mm:PinHeader_1x02_P2.54mm_Vertical, F.Cu at (129.2, 48.7)
- added J8: Limit Switch, Connector_PinHeader_2.54mm:PinHeader_1x04_P2.54mm_Vertical, F.Cu at (165.5, 61.9)
- added J9: Limit Switch, Connector_PinHeader_2.54mm:PinHeader_1x02_P2.54mm_Vertical, F.Cu at (138.1, 48.7)
- added R1: 10K, Resistor_SMD:R_1206_3216Metric_Pad1.30x1.75mm_HandSolder, F.Cu at (152.8, 104.1)
- added R10: 10k, Resistor_SMD:R_1206_3216Metric_Pad1.30x1.75mm_HandSolder, F.Cu at (138.0, 43.5)
- added R11: 10K, Resistor_SMD:R_1206_3216Metric_Pad1.30x1.75mm_HandSolder, F.Cu at (119.3, 53.1)
- added R12: 100, Resistor_SMD:R_1206_3216Metric_Pad1.30x1.75mm_HandSolder, F.Cu at (121.6, 53.1)
- added R15: 10K, Resistor_SMD:R_1206_3216Metric_Pad1.30x1.75mm_HandSolder, F.Cu at (175.7, 80.4)
- added R2: 10K, Resistor_SMD:R_1206_3216Metric_Pad1.30x1.75mm_HandSolder, F.Cu at (152.8, 33.1)
- added R25: 10K, Resistor_SMD:R_1206_3216Metric_Pad1.30x1.75mm_HandSolder, F.Cu at (152.8, 80.5)
- added R26: 10K, Resistor_SMD:R_1206_3216Metric_Pad1.30x1.75mm_HandSolder, F.Cu at (175.7, 56.8)
- added R27: 10K, Resistor_SMD:R_1206_3216Metric_Pad1.30x1.75mm_HandSolder, F.Cu at (152.8, 56.8)
- added R28: 10K, Resistor_SMD:R_1206_3216Metric_Pad1.30x1.75mm_HandSolder, F.Cu at (128.2, 53.1)
- added R29: 100, Resistor_SMD:R_1206_3216Metric_Pad1.30x1.75mm_HandSolder, F.Cu at (130.5, 53.1)
- added R3: 10K, Resistor_SMD:R_1206_3216Metric_Pad1.30x1.75mm_HandSolder, F.Cu at (175.7, 33.1)
- added R30: 10K, Resistor_SMD:R_1206_3216Metric_Pad1.30x1.75mm_HandSolder, F.Cu at (137.1, 53.0)
- added R31: 100, Resistor_SMD:R_1206_3216Metric_Pad1.30x1.75mm_HandSolder, F.Cu at (139.4, 53.1)
- added R32: 10K, Resistor_SMD:R_1206_3216Metric_Pad1.30x1.75mm_HandSolder, F.Cu at (119.3, 65.5)
- added R33: 10K, Resistor_SMD:R_1206_3216Metric_Pad1.30x1.75mm_HandSolder, F.Cu at (128.2, 65.7)
- added R34: 10K, Resistor_SMD:R_1206_3216Metric_Pad1.30x1.75mm_HandSolder, F.Cu at (137.1, 65.7)
- added R35: 100, Resistor_SMD:R_1206_3216Metric_Pad1.30x1.75mm_HandSolder, F.Cu at (121.6, 65.5)
- added R36: 100, Resistor_SMD:R_1206_3216Metric_Pad1.30x1.75mm_HandSolder, F.Cu at (130.5, 65.7)
- added R37: 100, Resistor_SMD:R_1206_3216Metric_Pad1.30x1.75mm_HandSolder, F.Cu at (139.4, 65.7)
- added R38: 100K, Resistor_SMD:R_1206_3216Metric_Pad1.30x1.75mm_HandSolder, F.Cu at (138.0, 38.7)
- added R39: 100, Resistor_SMD:R_1206_3216Metric_Pad1.30x1.75mm_HandSolder, F.Cu at (111.7, 88.5)
- added R40: 10K, Resistor_SMD:R_1206_3216Metric_Pad1.30x1.75mm_HandSolder, F.Cu at (113.2, 78.5)
- added R41: 10K, Resistor_SMD:R_1206_3216Metric_Pad1.30x1.75mm_HandSolder, F.Cu at (113.2, 81.0)
- added R8: 10K, Resistor_SMD:R_1206_3216Metric_Pad1.30x1.75mm_HandSolder, F.Cu at (175.7, 104.1)
- added SW1: SW_MEC_5E, Mylib:SW_B3F-1000, F.Cu at (111.2, 95.8)
- added U1: 3544-2, SamacSys_Parts:3544-2, F.Cu at (125.8, 40.5)
Routing:
- net +3V3: track 0.00 -> 403.9 mm, vias 0 -> 3
- net VPP: track 0.00 -> 305.6 mm, vias 0 -> 7
- net VSYS: track 0.00 -> 82.2 mm
- net DIR_8: track 0.00 -> 59.6 mm
- net STEP_8: track 0.00 -> 58.7 mm
- net IO27: track 0.00 -> 56.6 mm, vias 0 -> 1
- net IO28: track 0.00 -> 53.8 mm, vias 0 -> 1
- net DIR_5: track 0.00 -> 49.4 mm
- net STEP_5: track 0.00 -> 48.6 mm
- net LIMIT_SW_1: track 0.00 -> 46.9 mm, vias 0 -> 2
- net LIMIT_SW_3: track 0.00 -> 46.1 mm, vias 0 -> 2
- net LIMIT_SW_4: track 0.00 -> 41.8 mm, vias 0 -> 2
- net LIMIT_SW_2: track 0.00 -> 41.3 mm, vias 0 -> 2
- net DIR_3: track 0.00 -> 39.7 mm
- net STEP_3: track 0.00 -> 39.1 mm
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- added copper zone on B.Cu, net +12V
- added copper zone on B.Cu, net GND
- added copper zone on F.Cu, net GND
- added copper zone on In1.Cu, net GND
- added copper zone on In2.Cu, net GND
- added copper zone on B.Cu, net VPP
- added copper zone on F.Cu, net VPP
Other:
- board outline added: 90.2 x 98 mm
- copper layers 2 -> 4
- board text added: "CircuitScout Control V2"
- board text added: "Fangzheng Liu | fzliu@mit.edu"
- board text added: "RST"
