File: PCBPT_V2/Hardware/RPi_Pico_W_A4988_control_board/pico.kicad_sch (KiCad schematic)
At the start: 7 parts, among them IC2 RASPBERRY_PI_PICO_W, SW1 SW_MEC_5E

Commit message: udated by FZ
Parts:
- added J22: Limit Switch, Connector_PinHeader_2.54mm:PinHeader_1x02_P2.54mm_Vertical, symbol Connector:Conn_01x02_Male
- C2: footprint Capacitor_SMD:C_0603_1608Metric_Pad1.08x0.95mm_HandSolder -> Capacitor_SMD:C_1206_3216Metric_Pad1.33x1.80mm_HandSolder
- D2: footprint Diode_SMD:D_0603_1608Metric_Pad1.05x0.95mm_HandSolder -> Diode_SMD:D_0805_2012Metric_Pad1.15x1.40mm_HandSolder
- IC2: footprint RASPBERRYPIPICOW -> SamacSys_Parts:RASPBERRYPIPICOW
- R39, R40, R41: footprint Resistor_SMD:R_0603_1608Metric_Pad0.98x0.95mm_HandSolder -> Resistor_SMD:R_1206_3216Metric_Pad1.30x1.75mm_HandSolder
- SW1: footprint (none) -> Mylib:SW_B3F-1000
Connections:
- net IO18 is gone; now on net LIMIT_SW_3: IC2.24 (I2C1_SDA/_SPI0_SCK/GP18)
- net IO19 is gone; now on net LIMIT_SW_2: IC2.25 (I2C1_SCL/_SPI0_TX/GP19)
- net IO22 is gone; now on net LIMIT_SW_1: IC2.29 (GP22)
- net IO26 is gone; now on net LIMIT_SW_4: IC2.31 (I2C1_SDA/ADC0/GP26)
- net DIR_1: now also IC2.4 (I2C1_SDA_/SPI0_SCK/GP2); no longer IC2.2 (UART0_RX/I2C0_SCL_/SPI0_CSN/GP1)
- net DIR_2: now also IC2.1 (UART0_TX/I2C0_SDA_/SPI0_RX/GP0); no longer IC2.5 (I2C0_SCL_/SPI0_TX/GP3)
- net DIR_3: now also IC2.6 (UART1_TX/I2C0_SDA_/SPI0_RX/GP4); no longer IC2.7 (UART1_RX/I2C0_SCL_/SPI0_CSN/GP5)
- net DIR_4: now also IC2.9 (I2C1_SDA_/SPI0_SCK/GP6); no longer IC2.10 (I2C1_SCL_/SPI0_TX/GP7)
- net DIR_5: now also IC2.11 (UART1_TX/I2C0_SDA_/SPI1_RX/GP8); no longer IC2.12 (UART1_RX/I2C0_SCL_/SPI1_CSN/GP9)
- net DIR_6: now also IC2.14 (I2C1_SDA_/SPI1__SCK/GP10); no longer IC2.15 (I2C1_SCL_/SPI1__TX/GP11)
- net GND: now also J22.1 (Pin_1)
- net LIMIT_SW_1: no longer IC2.16 (UART0_TX/I2C0_SDA_/SPI1_RX_/GP12)
- net LIMIT_SW_2: no longer IC2.17 (UART0_RX/I2C0_SCL_/SPI1_CSN/GP13)
- net LIMIT_SW_3: no longer IC2.19 (I2C1_SDA/SPI1_SCK/GP14)
- net LIMIT_SW_4: no longer IC2.20 (I2C1_SCL/SPI1_TX/GP15)
- net STEP_1: now also IC2.5 (I2C0_SCL_/SPI0_TX/GP3); no longer IC2.1 (UART0_TX/I2C0_SDA_/SPI0_RX/GP0)
- net STEP_2: now also IC2.2 (UART0_RX/I2C0_SCL_/SPI0_CSN/GP1); no longer IC2.4 (I2C1_SDA_/SPI0_SCK/GP2)
- net STEP_3: now also IC2.7 (UART1_RX/I2C0_SCL_/SPI0_CSN/GP5); no longer IC2.6 (UART1_TX/I2C0_SDA_/SPI0_RX/GP4)
- net STEP_4: now also IC2.10 (I2C1_SCL_/SPI0_TX/GP7); no longer IC2.9 (I2C1_SDA_/SPI0_SCK/GP6)
- net STEP_5: now also IC2.12 (UART1_RX/I2C0_SCL_/SPI1_CSN/GP9); no longer IC2.11 (UART1_TX/I2C0_SDA_/SPI1_RX/GP8)
- net STEP_6: now also IC2.15 (I2C1_SCL_/SPI1__TX/GP11); no longer IC2.14 (I2C1_SDA_/SPI1__SCK/GP10)
- net at R39.2, SW1.3 (K), SW1.4 (A): now also J22.2 (Pin_2)
- new net DIR_7: IC2.19 (I2C1_SDA/SPI1_SCK/GP14)
- new net DIR_8: IC2.16 (UART0_TX/I2C0_SDA_/SPI1_RX_/GP12)
- new net STEP_7: IC2.20 (I2C1_SCL/SPI1_TX/GP15)
- new net STEP_8: IC2.17 (UART0_RX/I2C0_SCL_/SPI1_CSN/GP13)
Other:
- moved on the sheet: C2, D2, IC2, R39, SW1
