File: PCBPT_V2/Hardware/Board_To_Be_Tested/Board_To_Be_Tested.kicad_pcb (KiCad board)
At the start: 2 copper layers, 50 x 47 mm, 20 parts, among them U1 SHT15, U2 MOUDLE-SEEEDUINO-XIAO

Commit message: udated by FZ
Parts:
- added IC1: VEML7700-TR, SamacSys_Parts:VEML7700, F.Cu at (130.9, 77.4)
- added R10: 0, Resistor_SMD:R_1206_3216Metric_Pad1.30x1.75mm_HandSolder, F.Cu at (136.6, 85.8)
- added R8: 10k, Resistor_SMD:R_1206_3216Metric_Pad1.30x1.75mm_HandSolder, F.Cu at (132.4, 84.3)
- added R9: 10k, Resistor_SMD:R_1206_3216Metric_Pad1.30x1.75mm_HandSolder, F.Cu at (140.2, 79.4)
- moved C2 17.6 mm to (144.7, 90.4)
- moved D1 13.5 mm to (149.3, 89.1), turned to 90 degrees
- moved D2 4.14 mm to (144.7, 66.4)
- moved D3 4.14 mm to (144.7, 69.4)
- moved D4 4.14 mm to (144.7, 72.4)
- moved D5 4.14 mm to (144.7, 75.4)
- moved R1 4.14 mm to (150.7, 66.4)
- moved R2 4.14 mm to (150.7, 69.4)
- moved R3 4.14 mm to (150.7, 72.4)
- moved R6 4.14 mm to (150.7, 75.4)
- moved FID1 2.00 mm to (128.0, 67.0)
- moved FID2 2.00 mm to (172.0, 67.0)
- moved FID3 1.00 mm to (128.0, 105.0)
- moved FID4 1.00 mm to (172.0, 105.0)
Routing:
- net /SCL: track 0.00 -> 34.2 mm
- net /PWR: track 0.00 -> 33.1 mm
- net /SDA: track 0.00 -> 30.3 mm
- net VBUS: track 60.0 -> 40.9 mm
- net +3V3: track 71.9 -> 79.9 mm
- net GND: track 2.96 -> 7.87 mm
- net /DIN: track 17.1 -> 12.7 mm
- net /LED1: track 32.9 -> 31.7 mm
- net /LED4: track 18.2 -> 17.1 mm
- net /LED2: track 28.3 -> 27.4 mm
- net /LED3: track 23.0 -> 22.5 mm
Other:
- board size 50 x 47 mm -> 50 x 44 mm

Commit message: udated by FZ
Parts:
- added C3: 10uF, Capacitor_SMD:C_1206_3216Metric_Pad1.33x1.80mm_HandSolder, F.Cu at (132.0, 71.2)
Routing:
- net /PWR: track 33.1 -> 34.8 mm
Changed lines of the file:
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@@
     )
     (pad_to_mask_clearance 0)
-    (grid_origin 125 109)
+    (grid_origin 125 108)
     (pcbplotparams
       (layerselection 0x00010fc_ffffffff)
@@
     (fp_line (start 1.6 0.8) (end -1.6 0.8)
       (stroke (width 0.1) (type solid)) (layer "F.Fab"))
-    (pad "1" smd roundrect (at -1.55 0 90) (size 1.3 1.75) (layers "F.Cu" "F.Paste" "F.Mask") (roundrect_rratio 0.192308)
+    (pad "1" smd roundrect (at -1.55 0 90) (size 1.3 1.75) (layers "F.Cu" "F.Paste" "F.Mask") (roundrect_rratio 0.1923076923)
       (net 20 "/PWR") (pintype "passive"))
-    (pad "2" smd roundrect (at 1.55 0 90) (size 1.3 1.75) (layers "F.Cu" "F.Paste" "F.Mask") (roundrect_rratio 0.192308)
+    (pad "2" smd roundrect (at 1.55 0 90) (size 1.3 1.75) (layers "F.Cu" "F.Paste" "F.Mask") (roundrect_rratio 0.1923076923)
       (net 17 "/SCL") (pintype "passive"))
     (model "${KICAD6_3DMODEL_DIR}/Resistor_SMD.3dshapes/R_1206_3216Metric.wrl"
@@
       (net 10 "/LED2") (pintype "passive"))
     (model "${KICAD6_3DMODEL_DIR}/Resistor_SMD.3dshapes/R_1206_3216Metric.wrl"
+      (offset (xyz 0 0 0))
+      (scale (xyz 1 1 1))
+      (rotate (xyz 0 0 0))
+    )
+  )
+  (footprint "Capacitor_SMD:C_1206_3216Metric_Pad1.33x1.80mm_HandSolder" (layer "F.Cu")
+    (at 131.97 71.1975 -90)
+    (descr "Capacitor SMD 1206 (3216 Metric), square (rectangular) end terminal, IPC_7351 nominal with elongated pad for handsoldering. (Body size source: IPC-SM-782 page 76, https://www.pcb-3d.com/wordpress/wp-content/uploads/ipc-sm-782a_amendment_1_and_2.pdf), generated with kicad-footprint-generator")
+    (tags "capacitor handsolder")
+    (property "Sheetfile" "Board_To_Be_Tested.kicad_sch")
+    (property "Sheetname" "")
+    (property "ki_description" "Unpolarized capacitor, small symbol")
+    (property "ki_keywords" "capacitor cap")
+    (attr smd)
+    (fp_text reference "C3" (at 0 -1.85 90) (layer "F.SilkS") hide
+        (effects (font (size 1 1) (thickness 0.15)))
+    )
+    (fp_text value "10uF" (at 0 1.85 90) (layer "F.Fab")
+        (effects (font (size 1 1) (thickness 0.15)))
+    )
+    (fp_text user "${REFERENCE}" (at 0 0 90) (layer "F.Fab")
+        (effects (font (size 0.8 0.8) (thickness 0.12)))
+    )
+    (fp_line (start -0.711252 -0.91) (end 0.711252 -0.91)
+      (stroke (width 0.12) (type solid)) (layer "F.SilkS"))
+    (fp_line (start -0.711252 0.91) (end 0.711252 0.91)
+      (stroke (width 0.12) (type solid)) (layer "F.SilkS"))
+    (fp_line (start -2.48 -1.15) (end 2.48 -1.15)
+      (stroke (width 0.05) (type solid)) (layer "F.CrtYd"))
+    (fp_line (start -2.48 1.15) (end -2.48 -1.15)
+      (stroke (width 0.05) (type solid)) (layer "F.CrtYd"))
+    (fp_line (start 2.48 -1.15) (end 2.48 1.15)
+      (stroke (width 0.05) (type solid)) (layer "F.CrtYd"))
+    (fp_line (start 2.48 1.15) (end -2.48 1.15)
+      (stroke (width 0.05) (type solid)) (layer "F.CrtYd"))
+    (fp_line (start -1.6 -0.8) (end 1.6 -0.8)
+      (stroke (width 0.1) (type solid)) (layer "F.Fab"))
+    (fp_line (start -1.6 0.8) (end -1.6 -0.8)
+      (stroke (width 0.1) (type solid)) (layer "F.Fab"))
+    (fp_line (start 1.6 -0.8) (end 1.6 0.8)
+      (stroke (width 0.1) (type solid)) (layer "F.Fab"))
+    (fp_line (start 1.6 0.8) (end -1.6 0.8)
+      (stroke (width 0.1) (type solid)) (layer "F.Fab"))
+    (pad "1" smd roundrect (at -1.5625 0 270) (size 1.325 1.8) (layers "F.Cu" "F.Paste" "F.Mask") (roundrect_rratio 0.1886792453)
+      (net 1 "GND") (pintype "passive"))
+    (pad "2" smd roundrect (at 1.5625 0 270) (size 1.325 1.8) (layers "F.Cu" "F.Paste" "F.Mask") (roundrect_rratio 0.1886792453)
+      (net 20 "/PWR") (pintype "passive"))
+    (model "${KICAD6_3DMODEL_DIR}/Capacitor_SMD.3dshapes/C_1206_3216Metric.wrl"
       (offset (xyz 0 0 0))
       (scale (xyz 1 1 1))
@@
     (fp_line (start 1.6 0.8) (end -1.6 0.8)
       (stroke (width 0.1) (type solid)) (layer "F.Fab"))
-    (pad "1" smd roundrect (at -1.55 0 90) (size 1.3 1.75) (layers "F.Cu" "F.Paste" "F.Mask") (roundrect_rratio 0.192308)
+    (pad "1" smd roundrect (at -1.55 0 90) (size 1.3 1.75) (layers "F.Cu" "F.Paste" "F.Mask") (roundrect_rratio 0.1923076923)
       (net 18 "/SDA") (pintype "passive"))
-    (pad "2" smd roundrect (at 1.55 0 90) (size 1.3 1.75) (layers "F.Cu" "F.Paste" "F.Mask") (roundrect_rratio 0.192308)
+    (pad "2" smd roundrect (at 1.55 0 90) (size 1.3 1.75) (layers "F.Cu" "F.Paste" "F.Mask") (roundrect_rratio 0.1923076923)
       (net 20 "/PWR") (pintype "passive"))
     (model "${KICAD6_3DMODEL_DIR}/Resistor_SMD.3dshapes/R_1206_3216Metric.wrl"
@@
     (fp_line (start 1.6 0.8) (end -1.6 0.8)
       (stroke (width 0.1) (type solid)) (layer "F.Fab"))
-    (pad "1" smd roundrect (at -1.55 0) (size 1.3 1.75) (layers "F.Cu" "F.Paste" "F.Mask") (roundrect_rratio 0.192308)
+    (pad "1" smd roundrect (at -1.55 0) (size 1.3 1.75) (layers "F.Cu" "F.Paste" "F.Mask") (roundrect_rratio 0.1923076923)
       (net 20 "/PWR") (pintype "passive"))
-    (pad "2" smd roundrect (at 1.55 0) (size 1.3 1.75) (layers "F.Cu" "F.Paste" "F.Mask") (roundrect_rratio 0.192308)
+    (pad "2" smd roundrect (at 1.55 0) (size 1.3 1.75) (layers "F.Cu" "F.Paste" "F.Mask") (roundrect_rratio 0.1923076923)
       (net 13 "+3V3") (pintype "passive"))
     (model "${KICAD6_3DMODEL_DIR}/Resistor_SMD.3dshapes/R_1206_3216Metric.wrl"
@@
   (segment (start 140.21 77.83) (end 140.21 75.81) (width 0.508) (layer "F.Cu") (net 20))
   (segment (start 132.42 85.82) (end 132.4 85.84) (width 0.508) (layer "F.Cu") (net 20))
+  (segment (start 130.1 74.62) (end 130.11 74.62) (width 0.508) (layer "F.Cu") (net 20))
   (segment (start 130.1 74.62) (end 129.07 75.65) (width 0.508) (layer "F.Cu") (net 20))
+  (segment (start 131.97 72.93) (end 133.66 74.62) (width 0.508) (layer "F.Cu") (net 20))
   (segment (start 135 85.82) (end 132.42 85.82) (width 0.508) (layer "F.Cu") (net 20))
   (segment (start 133.66 74.62) (end 133.66 74.99) (width 0.508) (layer "F.Cu") (net 20))
   (segment (start 138.24 73.84) (end 134.44 73.84) (width 0.508) (layer "F.Cu") (net 20))
   (segment (start 133.66 74.99) (end 133.66 77.8) (width 0.508) (layer "F.Cu") (net 20))
+  (segment (start 131.97 72.76) (end 131.97 72.93) (width 0.508) (layer "F.Cu") (net 20))
   (segment (start 129.07 75.65) (end 129.07 84.33) (width 0.508) (layer "F.Cu") (net 20))
   (segment (start 134.44 73.84) (end 133.66 74.62) (width 0.508) (layer "F.Cu") (net 20))
   (segment (start 140.21 75.81) (end 138.24 73.84) (width 0.508) (layer "F.Cu") (net 20))
   (segment (start 129.07 84.33) (end 130.58 85.84) (width 0.508) (layer "F.Cu") (net 20))
-  (segment (start 133.66 74.62) (end 130.1 74.62) (width 0.508) (layer "F.Cu") (net 20))
+  (segment (start 130.11 74.62) (end 131.97 72.76) (width 0.508) (layer "F.Cu") (net 20))
   (zone (net 1) (net_name "GND") (layer "F.Cu") (hatch edge 0.5)
     (connect_pads (clearance 0.1524))
@@
     (polygon
       (pts
-        (xy 125 62)
-        (xy 175 62)
-        (xy 175 109)
-        (xy 125 109)
+        (xy 125.1 63.9)
+        (xy 175.1 63.9)
+        (xy 175 108)
+        (xy 125 108)
       )
     )

Commit message: udated by FZ
Parts:
- removed R10: 0, Resistor_SMD:R_1206_3216Metric_Pad1.30x1.75mm_HandSolder
Connections:
- C3 pad 2: /PWR -> +3V3
- IC1 pad 2: /PWR -> +3V3
- R8 pad 1: /PWR -> +3V3
- R9 pad 2: /PWR -> +3V3
Routing:
- net +3V3: track 79.9 -> 119.8 mm, vias 0 -> 2
- net /PWR: track 34.8 -> 0.00 mm
