File: PCBPT_V2/Hardware/Board_To_Be_Tested/Board_To_Be_Tested.kicad_sch (KiCad schematic)
At the start: 20 parts, among them U1 SHT15, U2 MOUDLE-SEEEDUINO-XIAO

Commit message: udated by FZ
Parts:
- added IC1: VEML7700-TR, SamacSys_Parts:VEML7700, symbol SamacSys_Parts:VEML7700-TR
- added R10: 0, Resistor_SMD:R_1206_3216Metric_Pad1.30x1.75mm_HandSolder, symbol Device:R_Small
- added R8, R9: 10k, Resistor_SMD:R_1206_3216Metric_Pad1.30x1.75mm_HandSolder, symbol Device:R_Small
Connections:
- net +3V3: now also R10.2
- net GND: now also IC1.3 (GND)
- net SCL: now also IC1.1 (SCL), R8.2
- net SDA: now also IC1.4 (SDA), R9.1
- new net PWR: IC1.2 (VDD), R10.1, R8.1, R9.2
- no-connect marks 1 -> 2
Other:
- moved on the sheet: C2, R4, R5, U2

Commit message: udated by FZ
Parts:
- added C3: 10uF, Capacitor_SMD:C_1206_3216Metric_Pad1.33x1.80mm_HandSolder, symbol Device:C_Small
Connections:
- net GND: now also C3.1
- net PWR: now also C3.2
Other:
- moved on the sheet: C2, D1, D2, D3, D4, D5, IC1, R1, R10, R2, R3, R4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

Commit message: udated by FZ
Parts:
- removed R10: 0, Resistor_SMD:R_1206_3216Metric_Pad1.30x1.75mm_HandSolder, symbol Device:R_Small
Connections:
- net PWR is gone; now on net +3V3: C3.2, IC1.2 (VDD), R8.1, R9.2
Changed lines of the file:
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@@
-    (stroke (width 0) (type default))
-  )
-  (wire (pts (xy 123.19 22.86) (xy 125.73 22.86))
     (stroke (width 0) (type default))
   )
@@
     (stroke (width 0) (type default))
   )
+  (wire (pts (xy 147.32 49.53) (xy 151.13 49.53))
+    (stroke (width 0) (type default))
+  )
   (wire (pts (xy 53.34 77.47) (xy 57.15 77.47))
     (stroke (width 0) (type default))
@@
     (stroke (width 0) (type default))
   )
-  (wire (pts (xy 130.81 22.86) (xy 132.08 22.86))
+  (wire (pts (xy 123.19 22.86) (xy 132.08 22.86))
     (stroke (width 0) (type default))
   )
@@
   )
   (label "LED1" (at 33.02 71.12 0) (fields_autoplaced)
-    (effects (font (size 1.27 1.27)) (justify left bottom))
-  )
-  (label "PWR" (at 137.16 22.86 0) (fields_autoplaced)
     (effects (font (size 1.27 1.27)) (justify left bottom))
   )
@@
   (label "A0" (at 80.01 41.91 180) (fields_autoplaced)
     (effects (font (size 1.27 1.27)) (justify right bottom))
-  )
-  (label "PWR" (at 147.32 49.53 0) (fields_autoplaced)
-    (effects (font (size 1.27 1.27)) (justify left bottom))
   )
   (label "SHT_DATA" (at 80.01 44.45 180) (fields_autoplaced)
@@
         (path "/7df7dad7-2f43-458c-9c95-c644d6c6fda5"
           (reference "#PWR0125") (unit 1)
-        )
-      )
-    )
-  )
-  (symbol (lib_id "Device:R_Small") (at 128.27 22.86 270) (unit 1)
-    (in_bom yes) (on_board yes) (dnp no)
-    (property "Reference" "R10" (at 128.27 25.4 90)
-      (effects (font (size 1.27 1.27)))
-    )
-    (property "Value" "0" (at 128.27 20.32 90)
-      (effects (font (size 1.27 1.27)))
-    )
-    (property "Footprint" "Resistor_SMD:R_1206_3216Metric_Pad1.30x1.75mm_HandSolder" (at 128.27 22.86 0)
-      (effects (font (size 1.27 1.27)) hide)
-    )
-    (property "Datasheet" "~" (at 128.27 22.86 0)
-      (effects (font (size 1.27 1.27)) hide)
-    )
-    (pin "1")
-    (pin "2")
-    (instances
-      (project "Board_To_Be_Tested"
-        (path "/24c45a69-1309-4a66-85dc-bd4044729c6d"
-          (reference "R10") (unit 1)
-        )
-      )
-      (project "feather_m0_bread"
-        (path "/7df7dad7-2f43-458c-9c95-c644d6c6fda5"
-          (reference "R6") (unit 1)
         )
       )
@@
         )
       )
+    )
+  )
+  (symbol (lib_id "power:+3V3") (at 151.13 49.53 0) (unit 1)
+    (in_bom yes) (on_board yes) (dnp no)
+    (property "Reference" "#PWR015" (at 151.13 53.34 0)
+      (effects (font (size 1.27 1.27)) hide)
+    )
+    (property "Value" "+3V3" (at 151.13 45.72 0)
+      (effects (font (size 1.27 1.27)))
+    )
+    (property "Footprint" "" (at 151.13 49.53 0)
+      (effects (font (size 1.27 1.27)) hide)
+    )
+    (property "Datasheet" "" (at 151.13 49.53 0)
+      (effects (font (size 1.27 1.27)) hide)
+    )
+    (pin "1")
+    (instances
+      (project "Board_To_Be_Tested"
+        (path "/24c45a69-1309-4a66-85dc-bd4044729c6d"
+          (reference "#PWR015") (unit 1)
+        )
+      )
+      (project "Cube_V1"
+        (path "/67ad53b0-e724-4354-8add-ffbe056bca93/07c0a6ff-eef2-4578-b5db-f7e0ea607e3d"
+          (reference "#PWR05") (unit 1)
+        )
+        (path "/67ad53b0-e724-4354-8add-ffbe056bca93/16e69528-41c2-4221-b894-390eb49a8b88"
+          (reference "#PWR010") (unit 1)
+        )
+      )
