File: PCBPT_V3/PCB/Board_To_Be_Tested_V2/Board_To_Be_Tested.kicad_pcb (KiCad board)
At the start: 2 copper layers, 50 x 44 mm, 24 parts, among them IC1 VEML7700-TR, U1 SHT15, U2 MOUDLE-SEEEDUINO-XIAO

Commit message: udated by FZ
Parts:
- removed R10: 0, Resistor_SMD:R_1206_3216Metric_Pad1.30x1.75mm_HandSolder
Routing:
- net /PWR: track 33.1 -> 12.9 mm
- net +3V3: track 79.9 -> 69.1 mm
Changed lines of the file:
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@@
     (fp_line (start 1.6 0.8) (end -1.6 0.8)
       (stroke (width 0.1) (type solid)) (layer "F.Fab"))
-    (pad "1" smd roundrect (at -1.55 0 90) (size 1.3 1.75) (layers "F.Cu" "F.Paste" "F.Mask") (roundrect_rratio 0.192308)
+    (pad "1" smd roundrect (at -1.55 0 90) (size 1.3 1.75) (layers "F.Cu" "F.Paste" "F.Mask") (roundrect_rratio 0.1923076923)
       (net 20 "/PWR") (pintype "passive"))
-    (pad "2" smd roundrect (at 1.55 0 90) (size 1.3 1.75) (layers "F.Cu" "F.Paste" "F.Mask") (roundrect_rratio 0.192308)
+    (pad "2" smd roundrect (at 1.55 0 90) (size 1.3 1.75) (layers "F.Cu" "F.Paste" "F.Mask") (roundrect_rratio 0.1923076923)
       (net 17 "/SCL") (pintype "passive"))
     (model "${KICAD6_3DMODEL_DIR}/Resistor_SMD.3dshapes/R_1206_3216Metric.wrl"
@@
     (fp_line (start 1.6 0.8) (end -1.6 0.8)
       (stroke (width 0.1) (type solid)) (layer "F.Fab"))
-    (pad "1" smd roundrect (at -1.55 0 90) (size 1.3 1.75) (layers "F.Cu" "F.Paste" "F.Mask") (roundrect_rratio 0.192308)
+    (pad "1" smd roundrect (at -1.55 0 90) (size 1.3 1.75) (layers "F.Cu" "F.Paste" "F.Mask") (roundrect_rratio 0.1923076923)
       (net 18 "/SDA") (pintype "passive"))
-    (pad "2" smd roundrect (at 1.55 0 90) (size 1.3 1.75) (layers "F.Cu" "F.Paste" "F.Mask") (roundrect_rratio 0.192308)
+    (pad "2" smd roundrect (at 1.55 0 90) (size 1.3 1.75) (layers "F.Cu" "F.Paste" "F.Mask") (roundrect_rratio 0.1923076923)
       (net 20 "/PWR") (pintype "passive"))
     (model "${KICAD6_3DMODEL_DIR}/Resistor_SMD.3dshapes/R_1206_3216Metric.wrl"
@@
     )
   )
-  (footprint "Resistor_SMD:R_1206_3216Metric_Pad1.30x1.75mm_HandSolder" (layer "F.Cu")
-    (at 136.55 85.82)
-    (descr "Resistor SMD 1206 (3216 Metric), square (rectangular) end terminal, IPC_7351 nominal with elongated pad for handsoldering. (Body size source: IPC-SM-782 page 72, https://www.pcb-3d.com/wordpress/wp-content/uploads/ipc-sm-782a_amendment_1_and_2.pdf), generated with kicad-footprint-generator")
-    (tags "resistor handsolder")
-    (property "Sheetfile" "Board_To_Be_Tested.kicad_sch")
-    (property "Sheetname" "")
-    (property "ki_description" "Resistor, small symbol")
-    (property "ki_keywords" "R resistor")
-    (attr smd)
-    (fp_text reference "R10" (at 0 -1.82) (layer "F.SilkS") hide
-        (effects (font (size 1 1) (thickness 0.15)))
-    )
-    (fp_text value "0" (at 0 1.82) (layer "F.Fab")
-        (effects (font (size 1 1) (thickness 0.15)))
-    )
-    (fp_text user "${REFERENCE}" (at 0 0) (layer "F.Fab")
-        (effects (font (size 0.8 0.8) (thickness 0.12)))
-    )
-    (fp_line (start -0.727064 -0.91) (end 0.727064 -0.91)
-      (stroke (width 0.12) (type solid)) (layer "F.SilkS"))
-    (fp_line (start -0.727064 0.91) (end 0.727064 0.91)
-      (stroke (width 0.12) (type solid)) (layer "F.SilkS"))
-    (fp_line (start -2.45 -1.12) (end 2.45 -1.12)
-      (stroke (width 0.05) (type solid)) (layer "F.CrtYd"))
-    (fp_line (start -2.45 1.12) (end -2.45 -1.12)
-      (stroke (width 0.05) (type solid)) (layer "F.CrtYd"))
-    (fp_line (start 2.45 -1.12) (end 2.45 1.12)
-      (stroke (width 0.05) (type solid)) (layer "F.CrtYd"))
-    (fp_line (start 2.45 1.12) (end -2.45 1.12)
-      (stroke (width 0.05) (type solid)) (layer "F.CrtYd"))
-    (fp_line (start -1.6 -0.8) (end 1.6 -0.8)
-      (stroke (width 0.1) (type solid)) (layer "F.Fab"))
-    (fp_line (start -1.6 0.8) (end -1.6 -0.8)
-      (stroke (width 0.1) (type solid)) (layer "F.Fab"))
-    (fp_line (start 1.6 -0.8) (end 1.6 0.8)
-      (stroke (width 0.1) (type solid)) (layer "F.Fab"))
-    (fp_line (start 1.6 0.8) (end -1.6 0.8)
-      (stroke (width 0.1) (type solid)) (layer "F.Fab"))
-    (pad "1" smd roundrect (at -1.55 0) (size 1.3 1.75) (layers "F.Cu" "F.Paste" "F.Mask") (roundrect_rratio 0.192308)
-      (net 20 "/PWR") (pintype "passive"))
-    (pad "2" smd roundrect (at 1.55 0) (size 1.3 1.75) (layers "F.Cu" "F.Paste" "F.Mask") (roundrect_rratio 0.192308)
-      (net 13 "+3V3") (pintype "passive"))
-    (model "${KICAD6_3DMODEL_DIR}/Resistor_SMD.3dshapes/R_1206_3216Metric.wrl"
-      (offset (xyz 0 0 0))
-      (scale (xyz 1 1 1))
-      (rotate (xyz 0 0 0))
-    )
-  )
   (footprint "Fiducial:Fiducial_1mm_Mask2mm" (layer "F.Cu")
     (at 128 105)
@@
   (segment (start 166.92075 98.37075) (end 166.92075 99.384) (width 0.508) (layer "F.Cu") (net 13))
   (segment (start 165.65 103.3) (end 166.92075 102.02925) (width 0.762) (layer "F.Cu") (net 13))
-  (segment (start 141.81 95.0625) (end 141.81 89.53) (width 0.508) (layer "F.Cu") (net 13))
   (segment (start 139.05 95.0625) (end 141.81 95.0625) (width 0.508) (layer "F.Cu") (net 13))
   (segment (start 139.05 100.75) (end 147.55 100.75) (width 0.508) (layer "F.Cu") (net 13))
@@
   (segment (start 139.0175 95.095) (end 139.05 95.0625) (width 0.508) (layer "F.Cu") (net 13))
   (segment (start 166.92075 102.02925) (end 166.92075 99.384) (width 0.762) (layer "F.Cu") (net 13))
-  (segment (start 141.81 89.53) (end 138.1 85.82) (width 0.508) (layer "F.Cu") (net 13))
   (segment (start 162.72 75.43) (end 152.2425 75.43) (width 0.508) (layer "F.Cu") (net 14))
   (segment (start 164.38075 81.384) (end 164.38075 77.09075) (width 0.508) (layer "F.Cu") (net 14))
@@
   (segment (start 161.84075 81.236761) (end 161.84075 81.384) (width 0.508) (layer "F.Cu") (net 18))
   (segment (start 136.2 77.8) (end 136.2 79.09) (width 0.508) (layer "F.Cu") (net 18))
-  (segment (start 130.58 85.84) (end 132.4 85.84) (width 0.508) (layer "F.Cu") (net 20))
   (segment (start 140.21 77.83) (end 140.21 75.81) (width 0.508) (layer "F.Cu") (net 20))
-  (segment (start 132.42 85.82) (end 132.4 85.84) (width 0.508) (layer "F.Cu") (net 20))
-  (segment (start 130.1 74.62) (end 129.07 75.65) (width 0.508) (layer "F.Cu") (net 20))
-  (segment (start 135 85.82) (end 132.42 85.82) (width 0.508) (layer "F.Cu") (net 20))
   (segment (start 133.66 74.62) (end 133.66 74.99) (width 0.508) (layer "F.Cu") (net 20))
   (segment (start 138.24 73.84) (end 134.44 73.84) (width 0.508) (layer "F.Cu") (net 20))
   (segment (start 133.66 74.99) (end 133.66 77.8) (width 0.508) (layer "F.Cu") (net 20))
-  (segment (start 129.07 75.65) (end 129.07 84.33) (width 0.508) (layer "F.Cu") (net 20))
   (segment (start 134.44 73.84) (end 133.66 74.62) (width 0.508) (layer "F.Cu") (net 20))
   (segment (start 140.21 75.81) (end 138.24 73.84) (width 0.508) (layer "F.Cu") (net 20))
-  (segment (start 129.07 84.33) (end 130.58 85.84) (width 0.508) (layer "F.Cu") (net 20))
-  (segment (start 133.66 74.62) (end 130.1 74.62) (width 0.508) (layer "F.Cu") (net 20))
   (zone (net 1) (net_name "GND") (layer "F.Cu") (hatch edge 0.5)
     (connect_pads (clearance 0.1524))
