File: PCBPT_V3/PCB/Probe/Probe.kicad_sch (KiCad schematic)
At the start: 52 parts, among them J1 Conn_01x02_Pin, J10 1_pin_sig, J11 1_pin_sig, J12 1_pin_sig, J13 1_pin_sig, J14 1_pin_sig, J15 Conn_01x04_Pin, J2 1_pin_sig, J3 USB_B_Micro, J4 1_pin_sig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

Commit message: udated by FZ
Parts:
- removed C1: 0.1uF, Capacitor_SMD:C_1206_3216Metric_Pad1.33x1.80mm_HandSolder, symbol Device:C_Small
- removed C10, C5, C6: 1uF, Capacitor_SMD:C_0603_1608Metric, symbol Device:C_Small
- removed C2: 0.1uF, Capacitor_SMD:C_0603_1608Metric, symbol Device:C_Small
- removed C3, C4: 22pF, Capacitor_SMD:C_0603_1608Metric, symbol Device:C_Small
- removed C7, C9: 10uF, Capacitor_SMD:C_0603_1608Metric, symbol Device:C_Small
- removed C8: 10uF, LED_SMD:LED_0805_2012Metric_Pad1.15x1.40mm_HandSolder, symbol Device:CP1_Small
- removed D1: SK6812, LED_SMD:LED_SK6812_PLCC4_5.0x5.0mm_P3.2mm, symbol LED:SK6812
- removed D2, D3, D4, D5, D6, D7, D8, D9: R, LED_SMD:LED_1206_3216Metric_Pad1.42x1.75mm_HandSolder, symbol Device:LED_Small_Filled
- removed FID1, FID2, FID3, FID4: Fiducial, Fiducial:Fiducial_1mm_Mask2mm, symbol Mechanical:Fiducial
- removed J10, J11, J12, J13, J14, J2, J4, J5, J6, J7, J8, J9: 1_pin_sig, symbol Mylib:1_pin_sig
- removed J15: Conn_01x04_Pin, symbol Connector:Conn_01x04_Pin
- removed J3: USB_B_Micro, Connector_USB:USB_Micro-B_Amphenol_10104110_Horizontal, symbol Connector:USB_B_Micro
- removed R1, R2, R3, R4, R5, R6, R8, R9: 200, Resistor_SMD:R_1206_3216Metric_Pad1.30x1.75mm_HandSolder, symbol Device:R_Small
- removed R7: 10k, Resistor_SMD:R_1206_3216Metric_Pad1.30x1.75mm_HandSolder, symbol Device:R_Small
- removed S1: tactile_switch, Button_Switch_SMD:SW_SPST_B3U-1000P, symbol dk_Tactile-Switches:B3U-1000P
- removed U1: SHT15, Mylib:DFN747X493X250-8N, symbol SHT15:SHT15
- removed U2: ATSAMD21G18A-AUT, Package_QFP:TQFP-48_7x7mm_P0.5mm, symbol MCU_Microchip_SAMD:ATSAMD21G18A-AUT
- removed U3: AP2112K-3.3, Package_TO_SOT_SMD:SOT-23-5_HandSoldering, symbol Regulator_Linear:AP2112K-3.3
- removed Y1: 32.768kHz, digikey-footprints:ECS-.327-12.5-34B-TR, symbol Device:Crystal_Small
- added H1, H2, H3: MountingHole, MountingHole:MountingHole_2.2mm_M2, symbol Mechanical:MountingHole
- added J2, J3: Conn_01x02_Pin, Connector_PinHeader_2.54mm:PinHeader_1x02_P2.54mm_Vertical, symbol Connector:Conn_01x02_Pin
- J1: footprint (none) -> Connector_PinHeader_2.54mm:PinHeader_1x02_P2.54mm_Horizontal
Connections:
- net SWDIO is gone; now on an unnamed net: J1.2 (Pin_2)
- net SWCLK: no longer names the net of J1.1 (Pin_1)
- net SWCLK: now also J2.1 (Pin_1), J2.2 (Pin_2), J3.1 (Pin_1), J3.2 (Pin_2)
- no-connect marks 3 -> 0

Commit message: udated by FZ
Parts:
- removed J2, J3: Conn_01x02_Pin, Connector_PinHeader_2.54mm:PinHeader_1x02_P2.54mm_Vertical, symbol Connector:Conn_01x02_Pin
Changed lines of the file:
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@@
 (kicad_sch (version 20230121) (generator eeschema)
   (paper "User" 250.012 159.995)
-  (junction (at 114.3 64.77) (diameter 0) (color 0 0 0 0)
-  )
-  (junction (at 114.3 67.31) (diameter 0) (color 0 0 0 0)
-  )
-  (junction (at 133.35 71.12) (diameter 0) (color 0 0 0 0)
-  )
-  (junction (at 133.35 64.77) (diameter 0) (color 0 0 0 0)
-  )
-  (junction (at 133.35 67.31) (diameter 0) (color 0 0 0 0)
-  )
-  (wire (pts (xy 133.35 67.31) (xy 133.35 71.12))
-    (stroke (width 0) (type default))
-  )
-  (wire (pts (xy 133.35 71.12) (xy 133.35 73.66))
-    (stroke (width 0) (type default))
-  )
-  (wire (pts (xy 133.35 64.77) (xy 133.35 67.31))
-    (stroke (width 0) (type default))
-  )
   (wire (pts (xy 114.3 64.77) (xy 114.3 67.31))
-    (stroke (width 0) (type default))
-  )
-  (wire (pts (xy 114.3 64.77) (xy 133.35 64.77))
-    (stroke (width 0) (type default))
-  )
-  (wire (pts (xy 114.3 67.31) (xy 133.35 67.31))
     (stroke (width 0) (type default))
   )
@@
     )
   )
-  (symbol (lib_id "Connector:Conn_01x02_Pin") (at 138.43 67.31 180) (unit 1)
-    (in_bom yes) (on_board yes) (dnp no) (fields_autoplaced)
-    (property "Reference" "J2" (at 139.1412 65.016 0)
-      (effects (font (size 1.27 1.27)) (justify right))
-    )
-    (property "Value" "Conn_01x02_Pin" (at 139.1412 67.064 0)
-      (effects (font (size 1.27 1.27)) (justify right))
-    )
-    (property "Footprint" "Connector_PinHeader_2.54mm:PinHeader_1x02_P2.54mm_Vertical" (at 138.43 67.31 0)
-      (effects (font (size 1.27 1.27)) hide)
-    )
-    (property "Datasheet" "~" (at 138.43 67.31 0)
-      (effects (font (size 1.27 1.27)) hide)
-    )
-    (pin "1")
-    (pin "2")
-    (instances
-      (project "Probe"
-        (path "/24c45a69-1309-4a66-85dc-bd4044729c6d"
-          (reference "J2") (unit 1)
-        )
-      )
-    )
-  )
   (symbol (lib_id "Mechanical:MountingHole") (at 114.3 88.9 0) (unit 1)
     (in_bom yes) (on_board yes) (dnp no) (fields_autoplaced)
@@
         )
       )
-    )
-  )
-  (symbol (lib_id "Connector:Conn_01x02_Pin") (at 138.43 73.66 180) (unit 1)
-    (in_bom yes) (on_board yes) (dnp no) (fields_autoplaced)
-    (property "Reference" "J3" (at 139.1412 71.366 0)
-      (effects (font (size 1.27 1.27)) (justify right))
-    )
-    (property "Value" "Conn_01x02_Pin" (at 139.1412 73.414 0)
-      (effects (font (size 1.27 1.27)) (justify right))
-    )
-    (property "Footprint" "Connector_PinHeader_2.54mm:PinHeader_1x02_P2.54mm_Vertical" (at 138.43 73.66 0)
-      (effects (font (size 1.27 1.27)) hide)
-    )
-    (property "Datasheet" "~" (at 138.43 73.66 0)
-      (effects (font (size 1.27 1.27)) hide)
-    )
-    (pin "1")
-    (pin "2")
-    (instances
-      (project "Probe"
-        (path "/24c45a69-1309-4a66-85dc-bd4044729c6d"
-          (reference "J3") (unit 1)
-        )
-      )
